Commit message: fix: the physics catch up before a descent, and may run faster than the model to do so
A swing is passed through only into another swing: before a descent the
physical arm has to be at the top of it, or the pad came down wherever
the physics still were, into the cases beside the spot. The simulated
joints may now turn half again as fast as the model, so trailing it
through a swing is something they can make up.

Co-Authored-By: Claude Fable 5.1 <noreply@anthropic.com>

File: sim/arm.urdf (robot description, URDF)
Before this commit: robot arm, 6 links, 5 joints
Joints:
- joint elbow: limit lower=-0.2 upper=3.3 effort=20000 velocity=2 -> lower=-0.2 upper=3.3 effort=20000 velocity=3
- joint roll: limit effort=5000 velocity=2 -> effort=5000 velocity=3
- joint shoulder: limit lower=-1.6 upper=3.2 effort=20000 velocity=2 -> lower=-1.6 upper=3.2 effort=20000 velocity=3
- joint wrist: limit lower=-4.0 upper=2.0 effort=20000 velocity=2 -> lower=-4.0 upper=2.0 effort=20000 velocity=3
- joint yaw: limit effort=20000 velocity=1.2 -> effort=20000 velocity=1.8
